Commit message: [modify] origin of r joint

File: motoman_description/robots/sia5/sia5_basic.urdf.xacro (robot description, xacro)
@@ -79,5 +79,6 @@
     <inertia ixx="0.0108400832201" ixy="0" ixz="0"
              iyy="0.010708873981" iyz="0" izz="0.00140456861413"/>
-    <origin xyz="-0.06 0.134 0.017" rpy="${M_PI/2} 0 0"/>
+    <!-- <origin xyz="-0.06 0.134 0.017" rpy="${M_PI/2} 0 0"/> -->
+    <origin xyz="-0.06 0.134 -0.017" rpy="${M_PI/2} 0 0"/>
     <limit effort="30.0" lower="${joint_r_lower_limit}"
            upper="${joint_r_upper_limit}" velocity="${joint_r_velocity_limit}"/>
