Commit message: [modify] world frame position

File: motoman_description/robots/sia5/sia5.urdf.xacro (robot description, xacro)
@@ -4,5 +4,5 @@
   <xacro:include filename="$(find motoman_description)/robots/sia5/sia5_basic.urdf.xacro" />
   <xacro:root_link_v0 name="world">
-    <origin xyz="0 0 0" rpy="0 0 0"/>
+    <origin xyz="0 0 0.2" rpy="0 0 0"/>
   </xacro:root_link_v0>
 </robot>
